File: driver_RGB.kicad_pcb (KiCad board)
At the start: 2 copper layers, 61.5 x 20 mm, 33 parts, among them J1 OUT, J2 Jack-DC, Q1 MMBT3904LT1G, Q2 MMBT3904LT1G, Q3 MMBT3904LT1G, U1 NE555, U2 NE555, U3 NE555

Commit message: agregando esquematico pdf
Other:
- board size 61.5 x 20 mm -> 60 x 20 mm
